Commit message: fix: cmd_vel bridge, headless server mode, physics stability, full test pass
- Fix ros_gz_bridge: bridge /model/aspect_rover/cmd_vel (Gazebo topic)
  and remap to ROS /cmd_vel; was bridging wrong topic, rover couldn't move
- Switch gz sim to -s (server-only) to prevent Qt/OGRE GUI crash killing
  the physics server in headless container environments
- Add flat ground_plane to lunar world SDF; dartsim cannot use heightmap
  collision geometry, causing ODE assertion crashes on contact
- Fix chassis and wheel inertia tensors to physically correct values
  (box/cylinder formulas); eliminates near-singular LCP matrices
- Lower default spawn z from 0.5m to 0.05m to prevent large drop impacts
- Fix aspect_bringup/setup.py import order (flake8 I100/I201)
- T-D1 PASS: odometry x=0.508m after 5s at 0.2m/s cmd_vel
- T-D2 PASS: /goto_waypoint returns success=True, cmd_vel linear.x=0.2
- All 9 linter tests pass (1 skipped: copyright)
- Document results and known issues in .docs/TESTING.md

File: src/aspect_description/urdf/aspect_rover.urdf.xacro (robot description, xacro)
@@ -40,7 +40,8 @@
     <inertial>
       <mass value="${chassis_mass}"/>
-      <inertia ixx="0.0001" ixy="0.0" ixz="0.0"
-               iyy="0.0001" iyz="0.0"
-               izz="0.0001"/>
+      <!-- Box inertia: ixx=m(y²+z²)/12, iyy=m(x²+z²)/12, izz=m(x²+y²)/12 -->
+      <inertia ixx="0.000273" ixy="0.0" ixz="0.0"
+               iyy="0.000482" iyz="0.0"
+               izz="0.000542"/>
     </inertial>
   </link>
@@ -65,7 +66,8 @@
       <inertial>
         <mass value="${wheel_mass}"/>
-        <inertia ixx="0.000005" ixy="0.0" ixz="0.0"
-                 iyy="0.000005" iyz="0.0"
-                 izz="0.000009"/>
+        <!-- Cylinder inertia: ixx=iyy=m(3r²+h²)/12, izz=mr²/2 -->
+        <inertia ixx="0.0000030" ixy="0.0" ixz="0.0"
+                 iyy="0.0000030" iyz="0.0"
+                 izz="0.0000050"/>
       </inertial>
     </link>

Commit message: fix(aspect_description): add friction to auger_feed_joint to prevent free-fall
Without collision geometry the housing falls under gravity to the
upper limit (0.05m) at sim start.  Housing mass is 0.036 kg so
gravity force ≈ 0.35 N.  Set friction=2.0 N (>> 0.35 N) and
damping=5.0 Ns/m to hold the joint retracted at position=0 until
an actuator command is applied (T-103).

File: src/aspect_description/urdf/aspect_rover.urdf.xacro (robot description, xacro)
@@ -218,4 +218,7 @@
     <limit lower="0" upper="${auger_feed_travel}"
            effort="50.0" velocity="0.01"/>
+    <!-- Friction >> gravity force on housing (0.036 kg × 9.81 ≈ 0.35 N) so
+         the joint stays retracted at sim start without an active controller. -->
+    <dynamics damping="5.0" friction="2.0"/>
   </joint>
   <!-- Auger bit — rotates within housing -->
